File: hardware/RP-ROM.kicad_pcb (KiCad board)
At the start: 2 copper layers, 19.2 x 37.1 mm, 34 parts, among them IC1 RP2354A, J1 Conn_01x14_Pin, J2 Conn_01x14_Pin, J3 Conn_01x03, J4 USB_C_Receptacle_USB2.0_16P, SW1 SW_Push, U1 RT9080-33GJ5, U2 CH213K, Y1 12m

Commit message: Rev2
Parts:
- C14: renamed from C13; footprint Capacitor_SMD:C_0201_0603Metric -> Capacitor_SMD:C_0402_1005Metric
- C4: renamed from C14; footprint Capacitor_SMD:C_0201_0603Metric -> Capacitor_SMD:C_0402_1005Metric
- C6: renamed from C11; footprint Capacitor_SMD:C_0201_0603Metric -> Capacitor_SMD:C_0402_1005Metric
- C7: renamed from C12; footprint Capacitor_SMD:C_0201_0603Metric -> Capacitor_SMD:C_0402_1005Metric
- R4: renamed from R9; value 470 -> 1k
- moved R5 0.27 mm to (72.7, 103.2)
- moved C4 0.15 mm to (70.9, 106.9)
- moved C14 0.15 mm to (72.1, 104.1)
- renumbered C4 to C10, C6 to C11, C9 to C12, C10 to C13, C7 to C5, C5 to C9, J4 to J1, J1 to J2, J2 to J3, J3 to J4, R8 to R5, R7 to R6, R4 to R7, R5 to R8, R6 to R9, U2 to U1, U1 to U2
Routing:
- net Net-(R5-Pad2): track 16.4 -> 17.1 mm
- net /A3: track 8.05 -> 7.54 mm
- net GND: track 0.90 -> 1.13 mm, vias 28 -> 39
Other:
- board text added: "RP-ROM Rev.2"
- board text removed: "RP-ROM Rev.1"

Commit message: Rev3
Parts:
- removed the U1 at (79.0, 95.1)
- added D1: RB521S-30, Diode_SMD:D_SOD-523, F.Cu at (78.6, 95.8)
- added D2: RB521S-30, Diode_SMD:D_SOD-523, F.Cu at (78.6, 94.3)
- renumbered D1 to D3, U2 to U1
Connections:
- J1 pad A4: +5V -> Net-(D2-A)
- J1 pad A9: +5V -> Net-(D2-A)
- J1 pad B4: +5V -> Net-(D2-A)
- J1 pad B9: +5V -> Net-(D2-A)
Routing:
- net Net-(D2-A): track 0.00 -> 12.5 mm
- net +5V: track 16.2 -> 3.66 mm
- net VCC: track 7.88 -> 8.91 mm, vias 1 -> 0
Other:
- board text added: "RP-ROM Rev.3"
- board text removed: "RP-ROM Rev.2"
