File: hardware/RP-ROM.kicad_sch (KiCad schematic)
At the start: 34 parts, among them IC1 RP2354A, J1 Conn_01x14_Pin, J2 Conn_01x14_Pin, J3 Conn_01x03, J4 USB_C_Receptacle_USB2.0_16P, SW1 SW_Push, U1 RT9080-33GJ5, U2 CH213K, Y1 12m

Commit message: Rev2
Parts:
- C1: JLCPCB Part # (none) -> C1538
- C10: renamed from C4; JLCPCB Part # (none) -> C23733
- C11: renamed from C6; JLCPCB Part # (none) -> C23733
- C12: renamed from C9; JLCPCB Part # (none) -> C1525
- C13: renamed from C10; JLCPCB Part # (none) -> C1525
- C14: renamed from C13; footprint Capacitor_SMD:C_0201_0603Metric -> Capacitor_SMD:C_0402_1005Metric; JLCPCB Part # (none) -> C1525
- C2, C3: JLCPCB Part # (none) -> C52923
- C4: renamed from C14; footprint Capacitor_SMD:C_0201_0603Metric -> Capacitor_SMD:C_0402_1005Metric; JLCPCB Part # (none) -> C1525
- C5: renamed from C7; JLCPCB Part # (none) -> C1548
- C6: renamed from C11; footprint Capacitor_SMD:C_0201_0603Metric -> Capacitor_SMD:C_0402_1005Metric; JLCPCB Part # (none) -> C1525
- C7: renamed from C12; footprint Capacitor_SMD:C_0201_0603Metric -> Capacitor_SMD:C_0402_1005Metric; JLCPCB Part # (none) -> C1525
- C8: JLCPCB Part # (none) -> C1548
- C9: renamed from C5; JLCPCB Part # (none) -> C23733
- D1: JLCPCB Part # (none) -> C51933305
- IC1: JLCPCB Part # (none) -> C41378174
- J1: renamed from J4; JLCPCB Part # (none) -> C2843970
- J4: renamed from J3; JLCPCB Part # (none) -> C7430452
- L1: JLCPCB Part # (none) -> C42411119
- R1: JLCPCB Part # (none) -> C26083
- R2, R3: JLCPCB Part # (none) -> C25905
- R4: renamed from R9; value 470 -> 1k; JLCPCB Part # (none) -> C11702
- R5: renamed from R8; JLCPCB Part # (none) -> C11702
- R6: renamed from R7; JLCPCB Part # (none) -> C11702
- R7: renamed from R4; JLCPCB Part # (none) -> C25100
- R8: renamed from R5; JLCPCB Part # (none) -> C25100
- R9: renamed from R6; JLCPCB Part # (none) -> C25105
- SW1: JLCPCB Part # (none) -> C720477
- U1: renamed from U2; JLCPCB Part # (none) -> C5456874
- U2: renamed from U1; JLCPCB Part # (none) -> C7528830
- Y1: JLCPCB Part # (none) -> C9002
- renumbered J1 to J2, J2 to J3
Other:
- note added: "Connector"
- note added: "Microcontroller"
- note added: "Regulator"
- note added: "USB"
- moved on the sheet: C1, C10, C11, C12, C13, C14, C2, C3, C4, C5, C6, C7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

Commit message: Rev3
Parts:
- removed U1: CH213K, Package_TO_SOT_SMD:SOT-23-3, symbol Yamadori_KiCad_Library:CH213K
- added D1, D2: RB521S-30, Diode_SMD:D_SOD-523, symbol Device:D_Shockley
- renumbered D1 to D3, U2 to U1
Connections:
- net +5V: now also D1.1 (K), D2.1 (K); no longer J1.A4 (VBUS), J1.A9 (VBUS), J1.B4 (VBUS), J1.B9 (VBUS)
- net VCC: now also D1.2 (A)
- new net: D2.2 (A), J1.A4 (VBUS), J1.A9 (VBUS), J1.B4 (VBUS), J1.B9 (VBUS)
